File: hardware/Bot_Arena_contol/Bot_Arena_contol.kicad_sch (KiCad schematic)
At the start: 31 parts, among them U1 ESP32-DEVKIT-V1

Commit message: Add footprint cleanup.
Parts:
- removed J1, J4, J5: (no value), symbol Connector_Generic:Conn_01x05
- removed J2, J3, J7: (no value), symbol Connector_Generic:Conn_01x03
- removed J6: (no value), symbol Connector_Generic:Conn_01x04
- added H1, H2, H3, H4: MountingHole, MountingHole:MountingHole_3.2mm_M3, symbol Mechanical:MountingHole
- added J1, J2, J3, J4: 5Pin_5mm_plus_2.54_pin, footprints:5pin_5mmpitch_plus_2.54_combo, symbol symbols:5Pin_5mm_plus_2.54_pin
- added J5, J6, J7: 3Pin_5mm_plus_2.54_pin, footprints:3pin_5mmpitch_plus_2.54mm, symbol symbols:3Pin_5mm_plus_2.54_pin
- D1, D2: value (none) -> rLED; footprint (none) -> Resistor_THT:R_Axial_DIN0411_L9.9mm_D3.6mm_P7.62mm_Vertical
- D3: value (none) -> gLED; footprint (none) -> Resistor_THT:R_Axial_DIN0411_L9.9mm_D3.6mm_P7.62mm_Vertical
- D4: value (none) -> yLED; footprint (none) -> Resistor_THT:R_Axial_DIN0411_L9.9mm_D3.6mm_P7.62mm_Vertical
- D5: value (none) -> LED; footprint (none) -> Resistor_THT:R_Axial_DIN0411_L9.9mm_D3.6mm_P7.62mm_Vertical
- R1, R10, R11, R12, R13, R7, R8, R9: value (none) -> 10k; footprint (none) -> Resistor_THT:R_Axial_DIN0207_L6.3mm_D2.5mm_P10.16mm_Horizontal
- R2, R3, R4, R5, R6: value (none) -> 330; footprint (none) -> Resistor_THT:R_Axial_DIN0207_L6.3mm_D2.5mm_P10.16mm_Horizontal
- U1: footprint MODULE_ESP32_DEVKIT_V1 -> ESP32DK1:MODULE_ESP32_DEVKIT_V1; symbol Bot_Arena_contol-rescue:ESP32-DEVKIT-V1-ESP32-DEVKIT-V1 -> ESP32DK1:ESP32-DEVKIT-V1
Connections:
- net +12V: now also J1.1 (Pin_1), J2.1 (Pin_1), J7.3 (Pin_3)
- net +3V3: now also J4.1 (Pin_1), J5.1 (Pin_1), J6.1 (Pin_1)
- net +5V: now also J3.5 (Pin_5), J7.1 (Pin_1)
- net Dis_Serial_Tx: now also J3.2 (Pin_2)
- net Dis_serial_Rx: now also J3.3 (Pin_3)
- net GND: now also J3.1 (Pin_1), J7.2 (Pin_2)
- net G_End: now also J4.4 (Pin_4)
- net G_Pause: now also J4.3 (Pin_3)
- net G_Reset: now also J4.5 (Pin_5)
- net G_Start: now also J4.2 (Pin_2)
- net T_A_End: now also J6.3 (Pin_3)
- net T_A_Start: now also J6.2 (Pin_2)
- net T_B_End: now also J5.3 (Pin_3)
- net T_B_Start: now also J5.2 (Pin_2)
- net s_Green: now also J1.4 (Pin_4), J2.4 (Pin_4)
- net s_Horn: now also J1.5 (Pin_5), J2.5 (Pin_5)
- net s_Red_1: now also J1.2 (Pin_2)
- net s_Red_2: now also J2.2 (Pin_2)
- net s_Yellow: now also J1.3 (Pin_3), J2.3 (Pin_3)
Other:
- note added: "Arena Controls"
